Commit message: fix interger erorr in mirror and typo

File: logiee_vehicle_description/urdf/vehicle.xacro (robot description, xacro)
@@ -2,5 +2,5 @@
 <robot xmlns:xacro="http://ros.org/wiki/xacro">
   <!-- load parameter -->
-  <xacro:property name="vehicle_info" value="${load_yaml('$(find logiee_description)/config/vehicle_info.param.yaml')}"/>
+  <xacro:property name="vehicle_info" value="${load_yaml('$(find logiee_vehicle_description)/config/vehicle_info.param.yaml')}"/>
   <!-- vehicle body -->
   <link name="base_link">
